Commit message: updated

File: urdf/fish_hpurv_macro.urdf.xacro (robot description, xacro)
@@ -109,32 +109,5 @@
     <limit effort="10" velocity="10" lower="-0.785398" upper="0.785398"/>
   </joint>
-  <joint name="laser_joint" type="fixed">
-    <parent link="link_base"/>
-    <child link="laser_frame"/>
-    <origin xyz="0.0325815 0.0493006 0.02" rpy="0 0 0"/>
-  </joint>
-  <link name="laser_frame">
-    <inertial>
-      <origin xyz="0 0 0" rpy="0 0 0"/>
-      <mass value="0.1"/>
-      <inertia ixx="0.0001" ixy="0" ixz="0" iyy="0.0001" iyz="0" izz="0.0001"/>
-    </inertial>
-    <visual>
-      <origin xyz="0 0 0" rpy="0 0 0"/>
-      <geometry>
-        <cylinder radius="0.05" length="0.04"/>
-      </geometry>
-      <material name="red">
-        <color rgba="1 0 0 1"/>
-      </material>
-    </visual>
-    <collision>
-      <origin xyz="0 0 0" rpy="0 0 0"/>
-      <geometry>
-        <cylinder radius="0.05" length="0.04"/>
-      </geometry>
-    </collision>
-  </link>
-  <gazebo reference="laser_frame">
+  <gazebo reference="link_base">
     <material>Gazebo/Red</material>
     <sensor name="laser" type="ray">
@@ -164,32 +137,5 @@
     </sensor>
   </gazebo>
-  <joint name="imu_joint" type="fixed">
-    <parent link="link_base"/>
-    <child link="imu_link"/>
-    <origin xyz="0.0325815 0.0493006 0.02" rpy="0 0 0"/>
-  </joint>
-  <link name="imu_link">
-    <inertial>
-      <origin xyz="0 0 0" rpy="0 0 0"/>
-      <mass value="0.1"/>
-      <inertia ixx="0.000001" ixy="0" ixz="0" iyy="0.000001" iyz="0" izz="0.000001"/>
-    </inertial>
-    <visual>
-      <origin xyz="0 0 0" rpy="0 0 0"/>
-      <geometry>
-        <box size="0.01 0.01 0.01"/>
-      </geometry>
-      <material name="blue">
-        <color rgba="0 0 1 1"/>
-      </material>
-    </visual>
-    <collision>
-      <origin xyz="0 0 0" rpy="0 0 0"/>
-      <geometry>
-        <box size="0.01 0.01 0.01"/>
-      </geometry>
-    </collision>
-  </link>
-  <gazebo reference="imu_link">
+  <gazebo reference="link_base">
     <sensor name="imu_sensor" type="imu">
       <update_rate>50</update_rate>
@@ -235,5 +181,5 @@
       <fluid_density>1000</fluid_density>
       <link name="link_base">
-        <volume>0.0122</volume>
+        <volume>0.0120</volume>
         <center_of_volume>0.0325815 0.0493006 0.02</center_of_volume>
       </link>
@@ -255,5 +201,5 @@
       <parameters>$(find fish_hpurv)/config/my_controllers.yaml</parameters>
     </plugin>
-    <plugin name="caudal_force_plugin" filename="/home/uav/ros2_ws/install/fish_hpurv/lib/fish_hpurv/libCaudalForcePlugin.so"/>
+    <plugin name="caudal_force_plugin" filename="/home/lohithvarma2004/ros2_ws/install/fish_hpurv/lib/fish_hpurv/libCaudalForcePlugin.so"/>
   </gazebo>
   <ros2_control name="FishSim" type="system">

Commit message: updated

File: urdf/fish_hpurv_macro.urdf.xacro (robot description, xacro)
@@ -109,72 +109,4 @@
     <limit effort="10" velocity="10" lower="-0.785398" upper="0.785398"/>
   </joint>
-  <gazebo reference="link_base">
-    <material>Gazebo/Red</material>
-    <sensor name="laser" type="ray">
-      <pose>0 0 0 0 0 0</pose>
-      <visualize>true</visualize>
-      <update_rate>10</update_rate>
-      <ray>
-        <scan>
-          <horizontal>
-            <samples>360</samples>
-            <min_angle>-3.14</min_angle>
-            <max_angle>3.14</max_angle>
-          </horizontal>
-        </scan>
-        <range>
-          <min>0.3</min>
-          <max>12</max>
-        </range>
-      </ray>
-      <plugin name="laser_controller" filename="libgazebo_ros_laser.so">
-        <ros>
-          <argument>~/out:=/scan</argument>
-        </ros>
-        <output_type>sensor_msgs/LaserScan</output_type>
-        <frame_name>laser_frame</frame_name>
-      </plugin>
-    </sensor>
-  </gazebo>
-  <gazebo reference="link_base">
-    <sensor name="imu_sensor" type="imu">
-      <update_rate>50</update_rate>
-      <always_on>true</always_on>
-      <visualize>true</visualize>
-      <plugin name="imu_plugin" filename="libgazebo_ros_imu.so">
-        <ros>
-          <argument>~/out:=/imu/data</argument>
-        </ros>
-        <topicName>/imu/data</topicName>
-        <frameName>imu_link</frameName>
-      </plugin>
-    </sensor>
-  </gazebo>
-  <gazebo reference="link_base">
-    <sensor name="dvl_sensor" type="ray">
-      <pose>0.03 -0.085 -0.06  0  3.14 0</pose>
-      <visualize>true</visualize>
-      <update_rate>10</update_rate>
-      <ray>
-        <scan>
-          <horizontal>
-            <samples>4</samples>
-            <min_angle>0</min_angle>
-            <max_angle>6.28319</max_angle>
-          </horizontal>
-          <vertical>
-            <samples>1</samples>
-            <min_angle>1.2217</min_angle>
-            <max_angle>1.2217</max_angle>
-          </vertical>
-        </scan>
-        <range>
-          <min>0.1</min>
-          <max>100</max>
-        </range>
-      </ray>
-      <plugin name="custom_dvl_plugin" filename="libfish_dvl_plugin.so"/>
-    </sensor>
-  </gazebo>
   <gazebo>
     <plugin name="buoyancy_plugin" filename="libBuoyancyPlugin.so">
